File: schematic/lrima-main/lrima-main.kicad_pcb (KiCad board)
At the start: 2 copper layers, 33.5 x 78.3 mm, 41 parts, among them IC1 STCC4-D-R3, P1 2.54-1*3P母, SW3 MSK12C02, SW4 TS-1101-C-W, U1 TLC555CD, U2 NRF_RST, U3 ER10BGFBK, U4 5-146277-5, U5 SHT4x, Y1 32.768kHz

Commit message: fix(pcb): Changed ALIVE to LRIMa
Other:
- board text added: "LRIMa Culture"
- board text removed: "ALIVEculture"
Changed lines of the file:
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@@
 			(plot_on_all_layers_selection 0x00000000_00000000_00000000_00000000)
 			(disableapertmacros no)
-			(usegerberextensions no)
+			(usegerberextensions yes)
 			(usegerberattributes yes)
 			(usegerberadvancedattributes yes)
@@
 			(sketchdnponfab yes)
 			(crossoutdnponfab yes)
-			(subtractmaskfromsilk no)
+			(subtractmaskfromsilk yes)
 			(outputformat 1)
 			(mirror no)
@@
 	)
 	(gr_text "V3.6.0"
-		(at 159.875 108.775 270)
+		(at 159.5 109 270)
 		(layer "F.SilkS")
 		(effects
@@
 		)
 	)
-	(gr_text "ALIVEculture"
+	(gr_text "LRIMa Culture"
 		(at 161 94.975 270)
 		(layer "F.SilkS")
