File: schematic/lrima-main/lrima-main.kicad_sch (KiCad schematic)
At the start: 41 parts, among them IC1 STCC4-D-R3, P1 2.54-1*3P母, SW1 TS-1101-C-W, SW2 TS-1101-C-W, SW3 MSK12C02, SW4 TS-1101-C-W, U1 TLC555CD, U2 NRF_RST, U3 ER10BGFBK, U4 5-146277-5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

Commit message: Update for schematic bom
Parts:
- BT1, BT2: symbol serre-lrima-altium-import:root_0_BS-24-A1AJ008_ -> Device:Battery; MPN (none) -> C964814
- C1: symbol serre-lrima-altium-import:root_0_0603B104K500NT_C30926_ -> Device:C; MPN (none) -> C30926
- C10, C11: MPN (none) -> C45359931
- C2: symbol serre-lrima-altium-import:root_0_CC0603KRX7R9BB103_ -> Device:C; MPN (none) -> C100042
- C3: symbol serre-lrima-altium-import:root_1_0603B471K500NT_ -> Device:C; MPN (none) -> C45359952
- C4, C5, C8: MPN (none) -> C30926
- C9: MPN (none) -> C1691
- IC1: MPN (none) -> 1649-STCC4-D-R3CT-ND
- L1: MPN (none) -> C23377983
- LED1, LED2: symbol serre-lrima-altium-import:root_2_NCD0603R1_C84263_ -> Device:LED; MPN (none) -> C84263
- P1: symbol serre-lrima-altium-import:root_0_2.54-1*3P母_ -> Connector_Generic:Conn_01x03; MPN (none) -> C492411
- R1: symbol serre-lrima-altium-import:root_0_0603WAF1002T5E_ -> Device:R_US; MPN (none) -> C25804
- R2: symbol serre-lrima-altium-import:root_2_SCR0603F330R_ -> Device:R_US; MPN (none) -> C3016255
- R3: symbol serre-lrima-altium-import:root_2_0603WAF1601T5E_ -> Device:R_US; MPN (none) -> C22847
- R4, R5: symbol serre-lrima-altium-import:root_0_0603WAF4700T5E_ -> Device:R_US; MPN (none) -> C23179
- R6, R7: symbol Device:R -> Device:R_US; MPN (none) -> C25804
- SW1, SW2, SW4: symbol serre-lrima-altium-import:root_0_TS-1101-C-W_ -> Switch:SW_Push; MPN (none) -> C318938
- SW3: MPN (none) -> C431540
- U1: MPN (none) -> C1520195
- U2: MPN (none) -> C2845026
- U3: MPN (none) -> C5173327
- U4: symbol serre-lrima-altium-import:root_0_5-146277-5_ -> Connector_Generic:Conn_01x05; MPN (none) -> C124387
- U5: MPN (none) -> 1649-SHT40-AD1B-R2TR-ND
- Y1: MPN (none) -> 1908-Q0,032768-JTX310-12,5-20-T2-70K-LFCT-ND
Connections:
- net GND_HUM_ENABLE: now also C1.2, R2.1; no longer C1.1, R2.2
- net at U1.5 (CONT): now also C2.1; no longer C2.2
- net at C3.1, U1.2 (TRIG), U1.6 (THRES): now also R3.2; no longer R3.1
- net +3V renamed +3V0
- net +3V_S renamed BAT
- net GND renamed GNDREF
- net GNDREF: now also C1.1, C2.2; no longer C1.2, C2.1
- new net: R2.2, R3.1, U1.7 (DISCH)
Other:
- moved on the sheet: U4
