File: schematic/lrima-ground/lrima-ground.kicad_pcb (KiCad board)
At the start: 2 copper layers, 31.2 x 96.4 mm, 10 parts, among them J1 Finger Join

Commit message: fix(pcb): Changed ALIVE to LRIMa
Other:
- board text added: "LRIMa Culture"
- board text removed: "ALIVEculture"
Changed lines of the file:
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@@
 		(net 1)
-	)
-	(gr_poly
-		(pts
-			(xy 156.195211 31.03407) (xy 156.274004 31.148463) (xy 156.408787 31.232564) (xy 156.492853 31.256238)
-			(xy 156.579972 31.263242) (xy 156.663376 31.252895) (xy 156.742231 31.224482) (xy 156.75153 31.219631)
-			(xy 156.821087 31.171176) (xy 156.873981 31.104057) (xy 156.928903 30.935403) (xy 156.958012 30.588589)
-			(xy 156.962142 30.252187) (xy 156.960097 29.867821) (xy 156.947668 29.650697) (xy 156.915415 29.530202)
-			(xy 156.853899 29.435722) (xy 156.762369 29.337017) (xy 156.661776 29.298405) (xy 156.559378 29.293178)
-			(xy 156.424643 29.304939) (xy 156.331283 29.353525) (xy 156.263178 29.424757) (xy 156.199891 29.512134)
-			(xy 156.167205 29.629084) (xy 156.155446 29.850096) (xy 156.154934 30.249657) (xy 156.164446 30.692007)
-			(xy 156.185123 30.985334)
-		)
-		(stroke
-			(width 0)
-			(type default)
-		)
-		(fill yes)
-		(layer "F.SilkS")
-	)
-	(gr_poly
-		(pts
-			(xy 158.569845 37.305163) (xy 158.653751 37.445039) (xy 158.779378 37.534855) (xy 158.929804 37.564192)
-			(xy 159.005953 37.5536) (xy 159.079591 37.525612) (xy 159.196647 37.430838) (xy 159.268413 37.324516)
-			(xy 159.299772 37.196766) (xy 159.306569 36.991398) (xy 159.296691 36.777589) (xy 159.264109 36.623535)
-			(xy 159.229412 36.551571) (xy 159.18192 36.494631) (xy 159.038059 36.4111) (xy 158.946769 36.379444)
-			(xy 158.883562 36.371669) (xy 158.828378 36.389513) (xy 158.761158 36.434717) (xy 158.63039 36.567182)
-			(xy 158.593339 36.623651) (xy 158.562279 36.750524) (xy 158.544274 37.081676)
-		)
-		(stroke
-			(width 0)
-			(type default)
-		)
-		(fill yes)
-		(layer "F.SilkS")
-	)
-	(gr_poly
-		(pts
-			(xy 156.292546 38.397439) (xy 156.442744 38.547574) (xy 157.706417 38.547574) (xy 158.753396 38.53545)
-			(xy 158.981027 38.515906) (xy 159.094278 38.483471) (xy 159.16661 38.436685) (xy 159.224603 38.380209)
-			(xy 159.297206 38.243292) (xy 159.309933 38.166991) (xy 159.305978 38.089054) (xy 159.285105 38.011963)
-			(xy 159.247001 37.937659) (xy 159.188257 37.865218) (xy 159.108648 37.796438) (xy 158.998831 37.757151)
-			(xy 158.791785 37.734154) (xy 158.420486 37.71424) (xy 157.593598 37.701659) (xy 157.085489 37.71424)
-			(xy 156.551987 37.753676) (xy 156.393514 37.787239) (xy 156.288946 37.837512) (xy 156.244293 37.880643)
-			(xy 156.212325 37.934198) (xy 156.170877 38.087047) (xy 156.164883 38.221057) (xy 156.186159 38.273652)
-			(xy 156.229414 38.33101)
-		)
-		(stroke
-			(width 0)
-			(type default)
-		)
-		(fill yes)
-		(layer "F.SilkS")
-	)
-	(gr_poly
-		(pts
-			(xy 156.29758 40.437758) (xy 156.421619 40.519521) (xy 156.755725 40.663805) (xy 157.943042 41.08975)
-			(xy 158.750986 41.355496) (xy 158.931494 41.394237) (xy 159.016593 41.386693) (xy 159.093509 41.363613)
-			(xy 159.160981 41.326268) (xy 159.217348 41.276096) (xy 159.261011 41.214787) (xy 159.290819 41.143527)
-			(xy 159.306569 41.031551) (xy 159.296256 40.923714) (xy 159.257633 40.833203) (xy 159.143172 40.726338)
-			(xy 158.892431 40.600537) (xy 158.447337 40.434385) (xy 158.023628 40.277618) (xy 157.805474 40.180827)
-			(xy 157.79704 40.171226) (xy 157.848746 40.144651) (xy 158.464958 39.913972) (xy 158.812029 39.784478)
-			(xy 159.074697 39.670494) (xy 159.210912 39.590085) (xy 159.284187 39.473349) (xy 159.309509 39.315077)
-			(xy 159.29851 39.231627) (xy 159.270761 39.154493) (xy 159.210912 39.073047) (xy 159.122992 39.003772)
-			(xy 159.031633 38.964388) (xy 158.870945 38.95968) (xy 158.607303 39.028916) (xy 158.533764 39.054491)
-			(xy 158.370758 39.112617) (xy 157.26086 39.50827) (xy 156.676748 39.724979) (xy 156.355973 39.868205)
-			(xy 156.270729 39.929998) (xy 156.209153 40.061363) (xy 156.20047 40.228139) (xy 156.220308 40.311282)
-			(xy 156.256378 40.386179)
-		)
-		(stroke
-			(width 0)
-			(type default)
-		)
-		(fill yes)
-		(layer "F.SilkS")
-	)
-	(gr_poly
-		(pts
-			(xy 158.644524 31.150467) (xy 158.771469 31.241922) (xy 158.919216 31.270965) (xy 158.995304 31.26068)
-			(xy 159.068849 31.233608) (xy 159.136268 31.190773) (xy 159.196647 31.131911) (xy 159.259841 31.044205)
-			(xy 159.292514 30.924947) (xy 159.304733 30.697677) (xy 159.306569 30.285925) (xy 159.297042 29.79378)
-			(xy 159.269355 29.51916) (xy 159.252028 29.464399) (xy 159.171428 29.371963) (xy 159.02556 29.301798)
-			(xy 158.936416 29.285738) (xy 158.847966 29.287749) (xy 158.785492 29.302456) (xy 158.667638 29.359429)
-			(xy 158.626295 29.400622) (xy 158.594885 29.457425) (xy 158.555755 29.646469) (xy 158.539637 30.281708)
-			(xy 158.553378 30.952677) (xy 158.584594 31.072131)
-		)
-		(stroke
-			(width 0)
-			(type default)
-		)
-		(fill yes)
-		(layer "F.SilkS")
-	)
-	(gr_poly
-		(pts
-			(xy 156.195211 34.162448) (xy 156.273759 34.275586) (xy 156.412548 34.363083) (xy 156.561056 34.391868)
-			(xy 156.706232 34.360697) (xy 157.5 34.098345) (xy 158.726755 33.658905) (xy 158.965487 33.566584)
-			(xy 159.133049 33.475816) (xy 159.207797 33.414185) (xy 159.259601 33.347366) (xy 159.303029 33.208953)
-			(xy 159.30573 33.149458) (xy 159.292784 33.04887) (xy 159.240243 32.961838) (xy 159.090415 32.855662)
-			(xy 158.713016 32.68889) (xy 158.089883 32.456137) (xy 158.084698 32.454251) (xy 157.135561 32.113603)
-			(xy 156.629559 31.961197) (xy 156.489315 31.944621) (xy 156.395748 31.961954) (xy 156.327492 32.008808)
-			(xy 156.263178 32.080799) (xy 156.250076 32.096471) (xy 156.186114 32.177179) (xy 156.160157 32.238021)
-			(xy 156.166074 32.311889) (xy 156.197728 32.431677) (xy 156.241707 32.538672) (xy 156.332695 32.627181)
-			(xy 156.564496 32.741994) (xy 157.145065 32.954619) (xy 157.719004 33.173918) (xy 157.088846 33.405025)
-			(xy 156.650891 33.561302) (xy 156.409599 33.660803) (xy 156.291655 33.739745) (xy 156.22374 33.834344)
-			(xy 156.169045 33.948069) (xy 156.16041 34.045857)
-		)
-		(stroke
-			(width 0)
-			(type default)
-		)
-		(fill yes)
-		(layer "F.SilkS")
 	)
 	(gr_line
@@
 			(type default)
 		)
-		(layer "F.SilkS")
-	)
-	(gr_poly
-		(pts
-			(xy 156.276603 35.687415) (xy 156.401628 35.827429) (xy 157.670336 35.840081) (xy 158.548173 35.839419)
-			(xy 158.997878 35.817264) (xy 159.050645 35.805499) (xy 159.161677 35.726148) (xy 159.265495 35.57424)
-			(xy 159.295664 35.49014) (xy 159.306569 35.408232) (xy 159.275678 35.285477) (xy 159.173302 35.14376)
-			(xy 159.099883 35.082933) (xy 159.017921 35.037955) (xy 158.865709 35.013603) (xy 158.223524 34.997387)
-			(xy 157.64852 35) (xy 156.401628 35.012652) (xy 156.276603 35.152665) (xy 156.211256 35.239302) (xy 156.170644 35.32419)
-			(xy 156.155559 35.39571) (xy 156.158408 35.467058) (xy 156.215591 35.607662)
-		)
-		(stroke
-			(width 0)
-			(type default)
-		)
-		(fill yes)
-		(layer "F.SilkS")
-	)
-	(gr_poly
-		(pts
-			(xy 157.470633 31.138659) (xy 157.604011 31.228635) (xy 157.759368 31.258757) (xy 157.83791 31.24926)
-			(xy 157.911525 31.223315) (xy 157.975308 31.182827) (xy 158.028802 31.127611) (xy 158.066389 31.064435)
-			(xy 158.090289 30.936024) (xy 158.112799 30.450355) (xy 158.110746 30.018261) (xy 158.092677 29.657906)
-			(xy 158.063871 29.49392) (xy 158.010361 29.411592) (xy 157.948008 29.352839) (xy 157.816495 29.30197)
-			(xy 157.729912 29.295708) (xy 157.600962 29.306047) (xy 157.504077 29.344684) (xy 157.460183 29.385367)
-			(xy 157.42501 29.442216) (xy 157.37522 29.626567) (xy 157.349057 30.014003) (xy 157.346447 30.300264)
-			(xy 157.346447 31.012984)
-		)
-		(stroke
-			(width 0)
-			(type default)
-		)
-		(fill yes)
 		(layer "F.SilkS")
 	)
@@
 		)
 	)
-	(gr_text "ALIVEculture"
-		(at 135 37 360)
+	(gr_text "LRIMa Culture"
+		(at 153 40 0)
 		(layer "F.SilkS")
 		(effects
@@
 		)
 	)
-	(group ""
-		(members "13c14d3e-b4ac-4317-99dc-5f66cf0b5694" "261381e1-1326-4409-94c7-e8b6b5a5933e"
-			"3f2ddad0-185c-4bbc-b505-51a2bf6afa24" "8c26503b-e5d1-4fef-8706-e255984c3c75"
-			"cc2c25c0-59fe-40e6-91fb-7a2a456b9b99" "d9feb033-3543-4abc-9d7e-bdf2d1fdabb7"
-			"ec3513de-f295-4006-aff1-cccd05fcf32f" "fbe33f30-4549-44f1-9893-c913f0b47dd4"
-		)
-	)

Commit message: Update for schematic bom
Connections:
- C1 pad 1: AOUT_GND_TEMP -> GNDREF
- C1 pad 2: GND -> AOUT_GND_TEMP
- C6 pad 1: GND -> AOUT_GND_HUM
- C6 pad 2: AOUT_GND_HUM -> GNDREF
- J1 pad 1: GND -> GNDREF
- J1 pad 3: GND -> GNDREF
- J1 pad 6: GND -> GNDREF
- J1 pad 7: GND -> GNDREF
- J1 pad 9: GND -> GNDREF
- R12 pad 1: GND -> GNDREF
- R13 pad 2: GND -> GNDREF
- R14 pad 2: GND -> GNDREF
Routing:
- net GND: track 111.5 -> 0.00 mm, vias 2 -> 0
- net (no net): track 0.00 -> 111.5 mm
- net GNDREF: vias 0 -> 2
- added copper zone on F.Cu, net AOUT_GND_TEMP
- added copper zone on B.Cu, net GNDREF
- removed copper zone on B.Cu, net GND
- removed copper zone on F.Cu, net GND
Changed lines of the file:
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@@
 	)
 	(net 0 "")
-	(net 1 "GND")
+	(net 1 "GNDREF")
 	(net 2 "IN_CLOCK_GND_HUM")
 	(net 3 "GROUND_TEMP_ENABLE")
@@
 			)
 		)
-		(property "Datasheet" "https://atta.szlcsc.com/upload/public/pdf/source/20180326/C100042_E8B0111D51DE3671A0A4A59FBCEFE81C.pdf"
+		(property "Datasheet" "~"
 			(at 0 0 0)
 			(layer "F.Fab")
@@
 			)
 		)
-		(property "Description" "Capacitance: Tolerance:±10% Tolerance:±10% Voltage Rated: Temperature Coefficient:"
+		(property "Description" "Unpolarized capacitor"
 			(at 0 0 0)
 			(layer "F.Fab")
@@
 			)
 		)
+		(property ki_fp_filters "C_*")
 		(sheetname "/")
 		(sheetfile "lrima-ground.kicad_sch")
@@
 			(layers "F.Cu" "F.Mask" "F.Paste")
 			(roundrect_rratio 0.25)
-			(net 5 "AOUT_GND_TEMP")
-			(pinfunction "1")
-			(pintype "input")
+			(net 1 "GNDREF")
+			(pintype "passive")
 		)
 		(pad "2" smd roundrect
@@
 			(layers "F.Cu" "F.Mask" "F.Paste")
 			(roundrect_rratio 0.25)
-			(net 1 "GND")
-			(pinfunction "2")
-			(pintype "input")
+			(net 5 "AOUT_GND_TEMP")
+			(pintype "passive")
 		)
 		(embedded_fonts no)
@@
 			(chamfer_ratio 0.2)
 			(chamfer)
-			(net 1 "GND")
+			(net 1 "GNDREF")
 			(pinfunction "Pin_1")
 			(pintype "passive")
@@
 			(chamfer_ratio 0.2)
 			(chamfer)
-			(net 1 "GND")
+			(net 1 "GNDREF")
 			(pinfunction "Pin_3")
 			(pintype "passive")
@@
 			(chamfer_ratio 0.2)
 			(chamfer)
-			(net 1 "GND")
+			(net 1 "GNDREF")
 			(pinfunction "Pin_6")
 			(pintype "passive")
@@
 			(chamfer_ratio 0.2)
 			(chamfer)
-			(net 1 "GND")
+			(net 1 "GNDREF")
 			(pinfunction "Pin_7")
 			(pintype "passive")
@@
 			(chamfer_ratio 0.2)
 			(chamfer)
-			(net 1 "GND")
+			(net 1 "GNDREF")
 			(pinfunction "Pin_9")
 			(pintype "passive")
@@
 			)
 		)
-		(property "Datasheet" "https://atta.szlcsc.com/upload/public/pdf/source/20220513/AD25F6E9AB017461977317CD0F039FBB.pdf"
+		(property "Datasheet" "http://www.vishay.com/docs/88503/1n4001.pdf"
 			(at 0 0 0)
 			(unlocked yes)
@@
 			)
 		)
-		(property "Description" "Power Dissipation: Reverse Voltage (Vr): Average Rectified Current (Io): Forward Voltage (Vf@If):1V@10mA Reverse Leakage Current:5uA@75V Reverse Recovery Time (trr): Operating Temperature:-65℃~+175℃@(Tj) Operating Temperature:-65℃~+175℃@(Tj)"
+		(property "Description" "1000V 1A General Purpose Rectifier Diode, DO-41"
 			(at 0 0 0)
 			(unlocked yes)
@@
 			)
 		)
+		(property "Sim.Device" "D"
+			(at 0 0 0)
+			(unlocked yes)
+			(layer "F.Fab")
+			(hide yes)
+			(effects
+				(font
+					(size 1 1)
+					(thickness 0.15)
+				)
+			)
+		)
+		(property "Sim.Pins" "1=K 2=A"
+			(at 0 0 0)
+			(unlocked yes)
+			(layer "F.Fab")
+			(hide yes)
+			(effects
+				(font
+					(size 1 1)
+					(thickness 0.15)
+				)
+			)
+		)
+		(property ki_fp_filters "D*DO?41*")
 		(sheetname "/")
 		(sheetfile "lrima-ground.kicad_sch")
@@
 			(net 4 "AOUT_GND_HUM")
 			(pinfunction "K")
-			(pintype "input")
+			(pintype "passive")
 		)
 		(pad "2" smd roundrect
@@
 			(net 2 "IN_CLOCK_GND_HUM")
 			(pinfunction "A")
-			(pintype "input")
+			(pintype "passive")
 		)
 		(embedded_fonts no)
@@
 			)
 		)
-		(property "Datasheet" "https://atta.szlcsc.com/upload/public/pdf/source/20161024/1477288428169.pdf"
+		(property "Datasheet" "~"
 			(at 0 0 0)
 			(layer "F.Fab")
@@
 			)
 		)
-		(property "Description" "Resistance @ 25°C: Resistance Tolerance: B Constant Tolerance: B Constant (25°C/50°C): Power: Steady State Current (Max):0.31mA B Constant (25°C/75°C):- B Constant (25°C/85°C):3334K B Constant (25°C/100°C):3455K Operating Temperature:-40°C~+125°C Operating Temperatu"
+		(property "Description" "Thermistor, temperature dependent resistor, US symbol"
 			(at 0 0 0)
 			(layer "F.Fab")
@@
 			)
 		)
+		(property ki_fp_filters "R_*")
 		(sheetname "/")
 		(sheetfile "lrima-ground.kicad_sch")
@@
 			(roundrect_rratio 0.25)
 			(net 5 "AOUT_GND_TEMP")
-			(pinfunction "1")
-			(pintype "input")
+			(pintype "passive")
 		)
 		(pad "2" smd roundrect
@@
 			(roundrect_rratio 0.25)
 			(net 3 "GROUND_TEMP_ENABLE")
-			(pinfunction "2")
-			(pintype "input")
+			(pintype "passive")
 		)
 		(embedded_fonts no)
@@
 			)
 		)
-		(property "Datasheet" "https://atta.szlcsc.com/upload/public/pdf/source/20200306/C422600_1E6D84923E4A46A82E41ADD87F860B5C.pdf"
+		(property "Datasheet" "~"
 			(at 0 0 0)
 			(layer "F.Fab")
@@
 			)
 		)
-		(property "Description" "Type:Thick Film Resistors Resistance: Tolerance:±1% Tolerance:±1% Power(Watts): Temperature Coefficient:±100ppm/℃ Temperature Coefficient:±100ppm/℃ Overload Voltage (Max): Operating Temperature Range:-55℃~+155℃ Operating Temperature Range:-55℃~+155℃"
+		(property "Description" "Resistor, US symbol"
 			(at 0 0 0)
 			(layer "F.Fab")
@@
 			)
 		)
+		(property ki_fp_filters "R_*")
 		(sheetname "/")
 		(sheetfile "lrima-ground.kicad_sch")
@@
 			(roundrect_rratio 0.25)
 			(net 4 "AOUT_GND_HUM")
-			(pinfunction "1")
-			(pintype "input")
+			(pintype "passive")
 		)
 		(pad "2" smd roundrect
@@
 			(layers "F.Cu" "F.Mask" "F.Paste")
 			(roundrect_rratio 0.25)
-			(net 1 "GND")
-			(pinfunction "2")
-			(pintype "input")
+			(net 1 "GNDREF")
+			(pintype "passive")
 		)
 		(embedded_fonts no)
@@
 			)
 		)
-		(property "Datasheet" "https://atta.szlcsc.com/upload/public/pdf/source/20200306/C422600_1E6D84923E4A46A82E41ADD87F860B5C.pdf"
+		(property "Datasheet" "~"
 			(at 0 0 0)
 			(layer "F.Fab")
@@
 			)
 		)
-		(property "Description" "Type:Thick Film Resistors Resistance: Tolerance:±1% Tolerance:±1% Power(Watts): Temperature Coefficient:±100ppm/℃ Temperature Coefficient:±100ppm/℃ Overload Voltage (Max): Operating Temperature Range:-55℃~+155℃ Operating Temperature Range:-55℃~+155℃"
+		(property "Description" "Resistor, US symbol"
 			(at 0 0 0)
 			(layer "F.Fab")
@@
 			)
 		)
+		(property ki_fp_filters "R_*")
 		(sheetname "/")
 		(sheetfile "lrima-ground.kicad_sch")
@@
 			(layers "F.Cu" "F.Mask" "F.Paste")
 			(roundrect_rratio 0.25)
-			(net 1 "GND")
-			(pinfunction "1")
-			(pintype "input")
+			(net 1 "GNDREF")
+			(pintype "passive")
 		)
 		(pad "2" smd roundrect
@@
 			(roundrect_rratio 0.25)
 			(net 5 "AOUT_GND_TEMP")
-			(pinfunction "2")
-			(pintype "input")
+			(pintype "passive")
 		)
 		(embedded_fonts no)
@@
 			)
 		)
-		(property "Datasheet" "https://atta.szlcsc.com/upload/public/pdf/source/20170420/1492670664651.pdf"
+		(property "Datasheet" "~"
 			(at 0 0 0)
 			(layer "F.Fab")
@@
 			)
 		)
-		(property "Description" "Capacitance: Tolerance:±10% Tolerance:±10% Voltage Rated: Temperature Coefficient:"
+		(property "Description" "Unpolarized capacitor"
 			(at 0 0 0)
 			(layer "F.Fab")
@@
 			)
 		)
+		(property ki_fp_filters "C_*")
 		(sheetname "/")
 		(sheetfile "lrima-ground.kicad_sch")
@@
 			(layers "F.Cu" "F.Mask" "F.Paste")
 			(roundrect_rratio 0.25)
-			(net 1 "GND")
-			(pinfunction "1")
-			(pintype "input")
+			(net 4 "AOUT_GND_HUM")
+			(pintype "passive")
 		)
 		(pad "2" smd roundrect
@@
 			(layers "F.Cu" "F.Mask" "F.Paste")
 			(roundrect_rratio 0.25)
-			(net 4 "AOUT_GND_HUM")
-			(pinfunction "2")
-			(pintype "input")
+			(net 1 "GNDREF")
+			(pintype "passive")
 		)
 		(embedded_fonts no)
@@
 			)
 		)
-		(property "Datasheet" "https://atta.szlcsc.com/upload/public/pdf/source/20200306/C422600_1E6D84923E4A46A82E41ADD87F860B5C.pdf"
+		(property "Datasheet" "~"
 			(at 0 0 90)
 			(layer "B.Fab")
@@
 			)
 		)
-		(property "Description" "Type:Thick Film Resistors Resistance: Tolerance:±1% Tolerance:±1% Power(Watts): Temperature Coefficient:±100ppm/℃ Temperature Coefficient:±100ppm/℃ Overload Voltage (Max): Operating Temperature Range:-55℃~+155℃ Operating Temperature Range:-55℃~+155℃"
+		(property "Description" "Resistor, US symbol"
 			(at 0 0 90)
 			(layer "B.Fab")
@@
 			)
 		)
+		(property ki_fp_filters "R_*")
 		(sheetname "/")
 		(sheetfile "lrima-ground.kicad_sch")
@@
 			(roundrect_rratio 0.25)
 			(net 6 "BOT_RESI")
-			(pinfunction "1")
-			(pintype "input")
+			(pintype "passive")
 		)
 		(pad "2" smd roundrect
@@
 			(layers "B.Cu" "B.Mask" "B.Paste")
 			(roundrect_rratio 0.25)
-			(net 1 "GND")
-			(pinfunction "2")
-			(pintype "input")
+			(net 1 "GNDREF")
+			(pintype "passive")
 		)
 		(embedded_fonts no)
@@
 		)
 		(layer "F.Cu")
-		(net 1)
 	)
 	(gr_line
@@
 		(width 0.381)
 		(layer "F.Cu")
-		(net 1)
+		(net 0)
 	)
 	(segment
@@
 		(width 0.381)
 		(layer "F.Cu")
-		(net 1)
+		(net 0)
 	)
 	(segment
@@
 		(width 4)
 		(layer "F.Cu")
-		(net 1)
+		(net 0)
 	)
 	(segment
@@
 		(width 4)
 		(layer "F.Cu")
-		(net 1)
+		(net 0)
 	)
 	(via
@@
 	)
 	(zone
-		(net 1)
-		(net_name "GND")
+		(net 5)
+		(net_name "AOUT_GND_TEMP")
 		(layer "F.Cu")
 		(hatch edge 0.5)
@@
 	(zone
 		(net 1)
-		(net_name "GND")
+		(net_name "GNDREF")
 		(layer "B.Cu")
 		(hatch edge 0.5)
