File: schematic/lrima-ground/lrima-ground.kicad_sch (KiCad schematic)
At the start: 10 parts, among them J1 Finger Join

Commit message: Update for schematic bom
Parts:
- C1: symbol ProDoc_Gro-easyedapro:CAP -> Device:C; MPN (none) -> C100042
- C6: symbol ProDoc_Gro-easyedapro:CAP -> Device:C; MPN (none) -> C100040
- D1: symbol ProDoc_Gro-easyedapro:D_1N4007 -> Diode:1N4007; MPN (none) -> C3011166
- R11: symbol ProDoc_Gro-easyedapro:NCP15XH103F03RC -> Device:Thermistor_US; MPN (none) -> C77131
- R12, R14: symbol ProDoc_Gro-easyedapro:Res -> Device:R_US; MPN (none) -> C25804
- R13: symbol ProDoc_Gro-easyedapro:Res -> Device:R_US; MPN (none) -> C22935
Connections:
- net AOUT_GND_HUM: now also C6.1; no longer C6.2
- net AOUT_GND_TEMP: now also C1.2; no longer C1.1
- net GND renamed GNDREF
- net GNDREF: now also C1.1, C6.2; no longer C1.2, C6.1
Other:
- moved on the sheet: R12, R13, R14
